Commit message: now it works using HOME sensors

File: head_meka_description/urdf/head_basic.urdf (robot description, URDF)
Before this commit: robot Robot1, 3 links, 2 joints
Joints:
- joint medium_to_upp: limit lower=-0.9 upper=0.9 effort=5 velocity=1 -> lower=-0.32 upper=0.62 effort=5 velocity=0.1
